File: pcbqa/samples/bench_bad.kicad_pcb (KiCad board)
At the start: 2 copper layers, 60 x 45 mm, 18 parts, among them J1 USB-C, J2 UART, U1 MCU32, U2 AP2112K-3.3, U3 24C16, Y1 12MHz

Commit message: Tezgah duzeltmesi: kilitli bilesenlere kusur ekilmiyor
Sorun: bench_bad'de J1/J2 hem harness tarafindan kilitli sayiliyor
(J/P/MH/H onekleri) hem de kart kenari kuralini ihlal ediyordu. Yerlestirici
onlari tasiyamadigi icin bu iki hata duzeltilemez bir cezaydi ve ulasilabilir
tavani 67'den 30'a dusuruyordu. Dort agent de bunu bagimsiz olarak buldu.

Duzeltme: kilitli bilesenler mekanik olarak sabittir, bu yuzden bench_good ile
AYNI (yasal) konumda duruyorlar. Fark yalnizca tasinabilir bilesenlerde.

Sonuc - hedef artik gercekten ulasilabilir:
  cluster  2 -> 67  (1 hata, HPWL 224)
  force    2 -> 67  (1 hata, HPWL 256)
  codex    2 -> 67  (1 hata, HPWL 261)
  anneal   2 -> 30  (3 hata, HPWL 444)  <- zayifligi artik izole

Ekilen kusur sayisi 9 -> 7 (ikisi kilitli bilesendeydi).
Belgelerdeki tezgah rakamlari guncellendi.
Parts:
- moved J1 6.40 mm to (8.00, 25.0)
- moved J2 4.60 mm to (34.0, 39.0)
Changed lines of the file:
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@@
 	(footprint "Gen:PinHeader_1x04"
 		(layer "F.Cu")
-		(at 1.6 25 90)
+		(at 8 25 90)
 		(property "Reference" "J1"
 			(at 0 -2.4 0)
@@
 	(footprint "Gen:PinHeader_1x04"
 		(layer "F.Cu")
-		(at 34 43.6)
+		(at 34 39)
 		(property "Reference" "J2"
 			(at 0 -2.4 0)
